File: Electrical/01b_V4 - Photoeye PCB/V1/00_Electrical/photoOnlyEyePCB_V1/PhotoeyeOnlyEye PCB_V1.kicad_pcb (KiCad board)
At the start: 2 copper layers, 20 x 20 mm, 4 parts, among them J1 B3B-PH-SM4-TB(LF)(SN), U2 RPR-220

Commit message: fixing the crossed wire for the photo sensor. deleting the old CNC jobs. Re-exporting gerbers and schematics. Re-mill with new files
Connections:
- U2 pad 3: /sensorValue -> +3.3V
- U2 pad 4: +3.3V -> /sensorValue
Routing:
- net +3.3V: track 20.3 -> 13.1 mm
- net /sensorValue: track 13.9 -> 11.4 mm
Changed lines of the file:
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@@
 			(layers "*.Cu" "*.Mask")
 			(remove_unused_layers no)
-			(net 3 "/sensorValue")
+			(net 2 "+3.3V")
 			(pinfunction "E")
 			(pintype "passive")
@@
 			(layers "*.Cu" "*.Mask")
 			(remove_unused_layers no)
-			(net 2 "+3.3V")
+			(net 3 "/sensorValue")
 			(pinfunction "C")
 			(pintype "passive")
@@
 	)
 	(segment
-		(start 121.5 98)
+		(start 124 98.3)
 		(end 121.5 100.8)
 		(width 0.5)
@@
 	)
 	(segment
-		(start 126 96.3)
-		(end 125 95.3)
+		(start 124 98)
+		(end 124 98.3)
+		(width 0.5)
+		(layer "F.Cu")
+		(net 2)
+	)
+	(segment
+		(start 124 96.552688)
+		(end 124 98)
 		(width 0.5)
 		(layer "F.Cu")
@@
 	(segment
 		(start 121.25 93.802687)
-		(end 121.25 89.9)
-		(width 0.5)
-		(layer "F.Cu")
-		(net 2)
-	)
-	(segment
-		(start 125 95.3)
-		(end 122.747313 95.3)
-		(width 0.5)
-		(layer "F.Cu")
-		(net 2)
-	)
-	(segment
-		(start 126 98.8)
-		(end 126 96.3)
-		(width 0.5)
-		(layer "F.Cu")
-		(net 2)
-	)
-	(segment
-		(start 122.860972 99.360972)
-		(end 125.439028 99.360972)
-		(width 0.5)
-		(layer "F.Cu")
-		(net 2)
-	)
-	(segment
-		(start 121.5 98)
-		(end 122.860972 99.360972)
-		(width 0.5)
-		(layer "F.Cu")
-		(net 2)
-	)
-	(segment
-		(start 122.747313 95.3)
+		(end 124 96.552688)
+		(width 0.5)
+		(layer "F.Cu")
+		(net 2)
+	)
+	(segment
+		(start 121.25 89.9)
 		(end 121.25 93.802687)
 		(width 0.5)
@@
 	)
 	(segment
-		(start 125.439028 99.360972)
-		(end 126 98.8)
-		(width 0.5)
-		(layer "F.Cu")
-		(net 2)
-	)
-	(segment
-		(start 122.4 96.4)
+		(start 119.5 96.4)
+		(end 119.9 96.4)
+		(width 0.5)
+		(layer "F.Cu")
+		(net 3)
+	)
+	(segment
+		(start 119.9 96.4)
+		(end 121.5 98)
+		(width 0.5)
+		(layer "F.Cu")
+		(net 3)
+	)
+	(segment
+		(start 119.5 96.4)
 		(end 117.25 96.4)
 		(width 0.5)
 		(layer "F.Cu")
-		(net 3)
-	)
-	(segment
-		(start 124 98)
-		(end 122.4 96.4)
-		(width 0.5)
-		(layer "F.Cu")

Commit message: updates and cnc files to photo eye pcbs
Changed lines of the file:
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@@
 		(pad "1" thru_hole circle
 			(at 0 0 180)
-			(size 1.62 1.62)
+			(size 2 2)
 			(drill 0.9)
 			(layers "*.Cu" "*.Mask")
@@
 		(pad "2" thru_hole circle
 			(at 5 -2.5 180)
-			(size 1.62 1.62)
+			(size 2 2)
 			(drill 0.9)
 			(layers "*.Cu" "*.Mask")
@@
 		(pad "3" thru_hole circle
 			(at 0 -5 180)
-			(size 1.62 1.62)
+			(size 2 2)
 			(drill 0.9)
 			(layers "*.Cu" "*.Mask")
@@
 		(pad "1" thru_hole rect
 			(at 0 0 90)
-			(size 1.416 1.416)
+			(size 2 2)
 			(drill 0.91)
 			(layers "*.Cu" "*.Mask")
@@
 		(pad "2" thru_hole circle
 			(at 0 2.5 90)
-			(size 1.416 1.416)
+			(size 2 2)
 			(drill 0.91)
 			(layers "*.Cu" "*.Mask")
@@
 		(pad "3" thru_hole circle
 			(at 2.8 2.5 90)
-			(size 1.416 1.416)
+			(size 2 2)
 			(drill 0.91)
 			(layers "*.Cu" "*.Mask")
@@
 		(pad "4" thru_hole circle
 			(at 2.8 0 90)
-			(size 1.416 1.416)
+			(size 2 2)
 			(drill 0.91)
 			(layers "*.Cu" "*.Mask")
