File: Electrical/01a_V4 Electrical Design/Connectors.kicad_sch (KiCad schematic)
At the start: 19 parts, among them J11 694106301002, J12 B2B-PH-SM4-TB(LF)(SN), J13 B3B-PH-SM4-TB(LF)(SN), J14 B2B-PH-SM4-TB(LF)(SN), J16 SSM-108-L-SV-K-TR, J18 B2B-PH-SM4-TB(LF)(SN), J3 B3B-PH-SM4-TB(LF)(SN), J8 B3B-PH-SM4-TB(LF)(SN), J9 B3B-PH-SM4-TB(LF)(SN), Q3 IRLML2502TRPBF, Q4 IRLML2502TRPBF

Commit message: updates to schematic to document outside components. Plans for additional electrical features requiring desiging a few more PCBs
Parts:
- renumbered H1 to H5, H2 to H7, J11 to J22, J16 to J24, J12 to J26, J13 to J27, J3 to J28, J8 to J30
Changed lines of the file:
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@@
 		(on_board yes)
 		(dnp no)
-		(property "Reference" "#PWR0131"
+		(property "Reference" "#PWR0212"
 			(at 93.98 143.51 0)
 			(effects
@@
 		)
 		(instances
-			(project "Animation Platter_V3"
-				(path "/6293f612-ad61-4760-ad66-c804a0624dd1/e7fa4b9b-7da5-430b-82c8-3eb99bf7d4d5"
-					(reference "#PWR0131")
+			(project ""
+				(path "/6293f612-ad61-4760-ad66-c804a0624dd1/e7fa4b9b-7da5-430b-82c8-3eb99bf7d4d5"
+					(reference "#PWR0212")
 					(unit 1)
 				)
@@
 		(dnp no)
 		(fields_autoplaced yes)
-		(property "Reference" "#PWR021"
+		(property "Reference" "#PWR0226"
 			(at 179.07 129.54 0)
 			(effects
@@
 		)
 		(instances
-			(project "Animation Platter_V3"
-				(path "/6293f612-ad61-4760-ad66-c804a0624dd1/e7fa4b9b-7da5-430b-82c8-3eb99bf7d4d5"
-					(reference "#PWR021")
+			(project ""
+				(path "/6293f612-ad61-4760-ad66-c804a0624dd1/e7fa4b9b-7da5-430b-82c8-3eb99bf7d4d5"
+					(reference "#PWR0226")
 					(unit 1)
 				)
@@
 		(dnp no)
 		(fields_autoplaced yes)
-		(property "Reference" "#PWR023"
+		(property "Reference" "#PWR0230"
 			(at 217.17 129.54 0)
 			(effects
@@
 		)
 		(instances
-			(project "Animation Platter_V3"
-				(path "/6293f612-ad61-4760-ad66-c804a0624dd1/e7fa4b9b-7da5-430b-82c8-3eb99bf7d4d5"
-					(reference "#PWR023")
+			(project ""
+				(path "/6293f612-ad61-4760-ad66-c804a0624dd1/e7fa4b9b-7da5-430b-82c8-3eb99bf7d4d5"
+					(reference "#PWR0230")
 					(unit 1)
 				)
@@
 		(on_board yes)
 		(dnp no)
-		(property "Reference" "H2"
+		(property "Reference" "H7"
 			(at 116.84 128.3278 0)
 			(effects
@@
 		)
 		(instances
-			(project "Animation Platter_V3"
-				(path "/6293f612-ad61-4760-ad66-c804a0624dd1/e7fa4b9b-7da5-430b-82c8-3eb99bf7d4d5"
-					(reference "H2")
+			(project ""
+				(path "/6293f612-ad61-4760-ad66-c804a0624dd1/e7fa4b9b-7da5-430b-82c8-3eb99bf7d4d5"
+					(reference "H7")
 					(unit 1)
 				)
@@
 		(on_board yes)
 		(dnp no)
-		(property "Reference" "#PWR080"
+		(property "Reference" "#PWR0227"
 			(at 185.42 80.01 0)
 			(effects
@@
 		)
 		(instances
-			(project "Animation Platter_V3"
-				(path "/6293f612-ad61-4760-ad66-c804a0624dd1/e7fa4b9b-7da5-430b-82c8-3eb99bf7d4d5"
-					(reference "#PWR080")
+			(project ""
+				(path "/6293f612-ad61-4760-ad66-c804a0624dd1/e7fa4b9b-7da5-430b-82c8-3eb99bf7d4d5"
+					(reference "#PWR0227")
 					(unit 1)
 				)
@@
 		(on_board yes)
 		(dnp no)
-		(property "Reference" "#PWR064"
+		(property "Reference" "#PWR0124"
 			(at 38.1 92.71 0)
 			(effects
@@
 		)
 		(instances
-			(project "Animation Platter_V3"
-				(path "/6293f612-ad61-4760-ad66-c804a0624dd1/e7fa4b9b-7da5-430b-82c8-3eb99bf7d4d5"
-					(reference "#PWR064")
+			(project ""
+				(path "/6293f612-ad61-4760-ad66-c804a0624dd1/e7fa4b9b-7da5-430b-82c8-3eb99bf7d4d5"
+					(reference "#PWR0124")
 					(unit 1)
 				)
@@
 		(on_board yes)
 		(dnp no)
-		(property "Reference" "J3"
+		(property "Reference" "J28"
 			(at 190.754 121.158 90)
 			(effects
@@
 		)
 		(instances
-			(project "Animation Platter_V3"
-				(path "/6293f612-ad61-4760-ad66-c804a0624dd1/e7fa4b9b-7da5-430b-82c8-3eb99bf7d4d5"
-					(reference "J3")
+			(project ""
+				(path "/6293f612-ad61-4760-ad66-c804a0624dd1/e7fa4b9b-7da5-430b-82c8-3eb99bf7d4d5"
+					(reference "J28")
 					(unit 1)
 				)
@@
 		(dnp no)
 		(fields_autoplaced yes)
-		(property "Reference" "#PWR077"
+		(property "Reference" "#PWR0225"
 			(at 179.07 69.85 0)
 			(effects
@@
 		)
 		(instances
-			(project "Animation Platter_V3"
-				(path "/6293f612-ad61-4760-ad66-c804a0624dd1/e7fa4b9b-7da5-430b-82c8-3eb99bf7d4d5"
-					(reference "#PWR077")
+			(project ""
+				(path "/6293f612-ad61-4760-ad66-c804a0624dd1/e7fa4b9b-7da5-430b-82c8-3eb99bf7d4d5"
+					(reference "#PWR0225")
 					(unit 1)
 				)
@@
 		(on_board yes)
 		(dnp no)
-		(property "Reference" "H1"
+		(property "Reference" "H5"
 			(at 96.52 128.3278 0)
 			(effects
@@
 			(project ""
 				(path "/6293f612-ad61-4760-ad66-c804a0624dd1/e7fa4b9b-7da5-430b-82c8-3eb99bf7d4d5"
-					(reference "H1")
+					(reference "H5")
 					(unit 1)
 				)
@@
 		(on_board yes)
 		(dnp no)
-		(property "Reference" "#PWR028"
+		(property "Reference" "#PWR0232"
 			(at 223.52 139.7 0)
 			(effects
@@
 		)
 		(instances
-			(project "Animation Platter_V3"
-				(path "/6293f612-ad61-4760-ad66-c804a0624dd1/e7fa4b9b-7da5-430b-82c8-3eb99bf7d4d5"
-					(reference "#PWR028")
+			(project ""
+				(path "/6293f612-ad61-4760-ad66-c804a0624dd1/e7fa4b9b-7da5-430b-82c8-3eb99bf7d4d5"
+					(reference "#PWR0232")
 					(unit 1)
 				)
@@
 		(on_board yes)
 		(dnp no)
-		(property "Reference" "#PWR0150"
+		(property "Reference" "#PWR0217"
 			(at 114.3 143.51 0)
 			(effects
@@
 		)
 		(instances
-			(project "Animation Platter_V3"
-				(path "/6293f612-ad61-4760-ad66-c804a0624dd1/e7fa4b9b-7da5-430b-82c8-3eb99bf7d4d5"
-					(reference "#PWR0150")
+			(project ""
+				(path "/6293f612-ad61-4760-ad66-c804a0624dd1/e7fa4b9b-7da5-430b-82c8-3eb99bf7d4d5"
+					(reference "#PWR0217")
 					(unit 1)
 				)
@@
 		(on_board yes)
 		(dnp no)
-		(property "Reference" "J8"
+		(property "Reference" "J30"
 			(at 228.854 121.158 90)
 			(effects
@@
 		)
 		(instances
-			(project "Animation Platter_V3"
-				(path "/6293f612-ad61-4760-ad66-c804a0624dd1/e7fa4b9b-7da5-430b-82c8-3eb99bf7d4d5"
-					(reference "J8")
+			(project ""
+				(path "/6293f612-ad61-4760-ad66-c804a0624dd1/e7fa4b9b-7da5-430b-82c8-3eb99bf7d4d5"
+					(reference "J30")
 					(unit 1)
 				)
@@
 		(on_board yes)
 		(dnp no)
-		(property "Reference" "#PWR065"
+		(property "Reference" "#PWR0211"
 			(at 72.39 92.71 0)
 			(effects
@@
 		)
 		(instances
-			(project "Animation Platter_V3"
-				(path "/6293f612-ad61-4760-ad66-c804a0624dd1/e7fa4b9b-7da5-430b-82c8-3eb99bf7d4d5"
-					(reference "#PWR065")
+			(project ""
+				(path "/6293f612-ad61-4760-ad66-c804a0624dd1/e7fa4b9b-7da5-430b-82c8-3eb99bf7d4d5"
+					(reference "#PWR0211")
 					(unit 1)
 				)
@@
 		(on_board yes)
 		(dnp no)
-		(property "Reference" "J13"
+		(property "Reference" "J27"
 			(at 190.754 61.468 90)
 			(effects
@@
 		)
 		(instances
-			(project "Animation Platter_V3"
-				(path "/6293f612-ad61-4760-ad66-c804a0624dd1/e7fa4b9b-7da5-430b-82c8-3eb99bf7d4d5"
-					(reference "J13")
+			(project ""
+				(path "/6293f612-ad61-4760-ad66-c804a0624dd1/e7fa4b9b-7da5-430b-82c8-3eb99bf7d4d5"
+					(reference "J27")
 					(unit 1)
 				)
@@
 		(on_board yes)
 		(dnp no)
-		(property "Reference" "J11"
+		(property "Reference" "J22"
 			(at 54.864 73.66 0)
 			(effects
@@
 		)
 		(instances
-			(project "Animation Platter_V3"
-				(path "/6293f612-ad61-4760-ad66-c804a0624dd1/e7fa4b9b-7da5-430b-82c8-3eb99bf7d4d5"
-					(reference "J11")
+			(project ""
+				(path "/6293f612-ad61-4760-ad66-c804a0624dd1/e7fa4b9b-7da5-430b-82c8-3eb99bf7d4d5"
+					(reference "J22")
 					(unit 1)
 				)
@@
 		(on_board yes)
 		(dnp no)
-		(property "Reference" "J12"
+		(property "Reference" "J26"
 			(at 151.892 121.158 90)
 			(effects
@@
 		)
 		(instances
-			(project "Animation Platter_V3"
-				(path "/6293f612-ad61-4760-ad66-c804a0624dd1/e7fa4b9b-7da5-430b-82c8-3eb99bf7d4d5"
-					(reference "J12")
+			(project ""
+				(path "/6293f612-ad61-4760-ad66-c804a0624dd1/e7fa4b9b-7da5-430b-82c8-3eb99bf7d4d5"
+					(reference "J26")
 					(unit 1)
 				)
@@
 		(on_board yes)
 		(dnp no)
-		(property "Reference" "#PWR022"
+		(property "Reference" "#PWR0228"
 			(at 185.42 139.7 0)
 			(effects
@@
 		)
 		(instances
-			(project "Animation Platter_V3"
-				(path "/6293f612-ad61-4760-ad66-c804a0624dd1/e7fa4b9b-7da5-430b-82c8-3eb99bf7d4d5"
-					(reference "#PWR022")
+			(project ""
+				(path "/6293f612-ad61-4760-ad66-c804a0624dd1/e7fa4b9b-7da5-430b-82c8-3eb99bf7d4d5"
+					(reference "#PWR0228")
 					(unit 1)
 				)
@@
 		(dnp no)
 		(fields_autoplaced yes)
-		(property "Reference" "#PWR088"
+		(property "Reference" "#PWR0222"
 			(at 144.78 129.54 0)
 			(effects
@@
 		)
 		(instances
-			(project "Animation Platter_V3"
-				(path "/6293f612-ad61-4760-ad66-c804a0624dd1/e7fa4b9b-7da5-430b-82c8-3eb99bf7d4d5"
-					(reference "#PWR088")
+			(project ""
+				(path "/6293f612-ad61-4760-ad66-c804a0624dd1/e7fa4b9b-7da5-430b-82c8-3eb99bf7d4d5"
+					(reference "#PWR0222")
 					(unit 1)
 				)
@@
 		(dnp no)
 		(fields_autoplaced yes)
-		(property "Reference" "#PWR0185"
+		(property "Reference" "#PWR0125"
 			(at 72.39 77.47 0)
 			(effects
@@
 			(project ""
 				(path "/6293f612-ad61-4760-ad66-c804a0624dd1/e7fa4b9b-7da5-430b-82c8-3eb99bf7d4d5"
-					(reference "#PWR0185")
+					(reference "#PWR0125")
 					(unit 1)
 				)
@@
 		(on_board yes)
 		(dnp no)
-		(property "Reference" "J16"
+		(property "Reference" "J24"
 			(at 117.348 100.076 90)
 			(effects
@@
 			(project ""
 				(path "/6293f612-ad61-4760-ad66-c804a0624dd1/e7fa4b9b-7da5-430b-82c8-3eb99bf7d4d5"
-					(reference "J16")
-					(unit 1)
-				)
+					(reference "J24")
+					(unit 1)
+				)

Commit message: main schematic tweaks. Started the 'Saber' PCB which is the new end effector for the strobe light. Schematic nearly finished. Need to create footprint for LEDs and layout the board to be CNC milled.
Other:
- note added: "Optional Sensor Pullups"
- note added: "add TVS diode add current limit resistor"
- note added: "add TVS diodes"
- note added: "add default state resistor add current limit resistor"
- note added: "extra sensor"
- note removed: "Extra Hall sensor"
- note removed: "Optional Hall Sensor Pullups"
- note removed: "Platter ID Hall sensor"
- note removed: "Platter Index Hall sensor"
- note removed: "add default state resistor"
- note removed: "add optional default state resistor"
- company: (none) -> Kadin Whiting
- title: (none) -> Connectors
