File: Electrical/01a_V4 Electrical Design/Display and LEDs.kicad_sch (KiCad schematic)
At the start: 20 parts, among them J1 B3B-PH-SM4-TB(LF)(SN), U2 74HC3G34DC

Commit message: main schematic tweaks. Started the 'Saber' PCB which is the new end effector for the strobe light. Schematic nearly finished. Need to create footprint for LEDs and layout the board to be CNC milled.
Other:
- company: (none) -> Kadin Whiting
- title: (none) -> Neopixels
