File: Electrical/01a_V4 Electrical Design/Interface.kicad_sch (KiCad schematic)
At the start: 40 parts, among them SW1 100SP1T1B4M2QE, SW2 100SP1T1B4M2QE, SW3 EN12-HS22AF20, SW4 100SP1T1B4M2QE

Commit message: main schematic tweaks. Started the 'Saber' PCB which is the new end effector for the strobe light. Schematic nearly finished. Need to create footprint for LEDs and layout the board to be CNC milled.
Other:
- company: (none) -> Kadin Whiting
- title: (none) -> Machine Interface
