File: Electrical/01a_V4 Electrical Design/Motor & LEDs_sch.kicad_sch (KiCad schematic)
At the start: 18 parts, among them J21 B2B-PH-SM4-TB(LF)(SN), J4 B2B-PH-SM4-TB(LF)(SN), J5 SSM-103-F-SV-P-TR, J6 1711725, J7 B4B-XH-A(LF)(SN), Q2 IRLML2502TRPBF

Commit message: updates to schematic to document outside components. Plans for additional electrical features requiring desiging a few more PCBs
Parts:
- J6: value 1711725 -> 1x2 5mm screw terminal; footprint Footprint drive Dump 1:1711725 -> (none)
Changed lines of the file:
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@@
 		(dnp no)
 		(property "Reference" "J6"
-			(at 116.332 135.128 90)
+			(at 112.014 129.032 90)
 			(effects
 				(font
@@
 			)
 		)
-		(property "Value" "1711725"
-			(at 108.712 131.826 90)
+		(property "Value" "1x2 5mm screw terminal"
+			(at 102.616 131.318 90)
 			(effects
 				(font
@@
 			)
 		)
-		(property "Footprint" "Footprint drive Dump 1:1711725"
+		(property "Footprint" ""
 			(at 111.76 134.62 0)
 			(effects
@@
 		)
 		(instances
-			(project "Animation Platter_V3"
+			(project ""
+				(path "/6293f612-ad61-4760-ad66-c804a0624dd1/0e41a5d4-74a8-4029-8d4e-febea7e98f25"
+					(reference "J6")
+					(unit 1)
+				)
 				(path "/6293f612-ad61-4760-ad66-c804a0624dd1/dd4c35ab-e025-4cfe-9a78-605a270d4a30"
 					(reference "J6")

Commit message: main schematic tweaks. Started the 'Saber' PCB which is the new end effector for the strobe light. Schematic nearly finished. Need to create footprint for LEDs and layout the board to be CNC milled.
Other:
- company: (none) -> Kadin Whiting
- title: (none) -> Motor and Strobe
