File: Electrical/01a_V4 Electrical Design/Power.kicad_sch (KiCad schematic)
At the start: 7 parts, among them K4 PR30-24V-450-1A-E, SW6 B2B-PH-SM4-TB(LF)(SN)

Commit message: main schematic tweaks. Started the 'Saber' PCB which is the new end effector for the strobe light. Schematic nearly finished. Need to create footprint for LEDs and layout the board to be CNC milled.
Other:
- company: (none) -> Kadin Whiting
- title: (none) -> Power
