File: Electrical/01a_V4 - Saber - Spot Light/V1/00_Electrical Design/Saber_V1/LEDs.kicad_sch (KiCad schematic)
At the start: 117 parts, among them J1 Conn_01x04

Commit message: designed the saber PCB, exported the files. Time to attempt to CNC and test it
Parts:
- D1, D10, D11, D12, D13, D14, D15, D16, D17, D18, D19, D2, D20, D21, D22, D3, D32, D4, D42, D43, D5, D53, D6, D63, D64, D7, D74, D8, D84, D9: footprint (none) -> Saber_V1:L1305095001400001
- D23: renamed from D29; footprint (none) -> Saber_V1:L1305095001400001
- D24: renamed from D36; footprint (none) -> Saber_V1:L1305095001400001
- D25: renamed from D23; footprint (none) -> Saber_V1:L1305095001400001
- D26: renamed from D30; footprint (none) -> Saber_V1:L1305095001400001
- D27: renamed from D37; footprint (none) -> Saber_V1:L1305095001400001
- D28: renamed from D24; footprint (none) -> Saber_V1:L1305095001400001
- D29: renamed from D31; footprint (none) -> Saber_V1:L1305095001400001
- D30: renamed from D38; footprint (none) -> Saber_V1:L1305095001400001
- D31: renamed from D25; footprint (none) -> Saber_V1:L1305095001400001
- D33: renamed from D39; footprint (none) -> Saber_V1:L1305095001400001
- D34: renamed from D26; footprint (none) -> Saber_V1:L1305095001400001
- D35: renamed from D33; footprint (none) -> Saber_V1:L1305095001400001
- D36: renamed from D40; footprint (none) -> Saber_V1:L1305095001400001
- D37: renamed from D27; footprint (none) -> Saber_V1:L1305095001400001
- D38: renamed from D34; footprint (none) -> Saber_V1:L1305095001400001
- D39: renamed from D41; footprint (none) -> Saber_V1:L1305095001400001
- D40: renamed from D28; footprint (none) -> Saber_V1:L1305095001400001
- D41: renamed from D35; footprint (none) -> Saber_V1:L1305095001400001
- D44: renamed from D50; footprint (none) -> Saber_V1:L1305095001400001
- D45: renamed from D57; footprint (none) -> Saber_V1:L1305095001400001
- D46: renamed from D44; footprint (none) -> Saber_V1:L1305095001400001
- D47: renamed from D51; footprint (none) -> Saber_V1:L1305095001400001
- D48: renamed from D58; footprint (none) -> Saber_V1:L1305095001400001
- D49: renamed from D45; footprint (none) -> Saber_V1:L1305095001400001
- D50: renamed from D52; footprint (none) -> Saber_V1:L1305095001400001
- D51: renamed from D59; footprint (none) -> Saber_V1:L1305095001400001
- D52: renamed from D46; footprint (none) -> Saber_V1:L1305095001400001
- D54: renamed from D60; footprint (none) -> Saber_V1:L1305095001400001
- D55: renamed from D47; footprint (none) -> Saber_V1:L1305095001400001
- D56: renamed from D54; footprint (none) -> Saber_V1:L1305095001400001
- D57: renamed from D61; footprint (none) -> Saber_V1:L1305095001400001
- D58: renamed from D48; footprint (none) -> Saber_V1:L1305095001400001
- D59: renamed from D55; footprint (none) -> Saber_V1:L1305095001400001
- D60: renamed from D62; footprint (none) -> Saber_V1:L1305095001400001
- D61: renamed from D49; footprint (none) -> Saber_V1:L1305095001400001
- D62: renamed from D56; footprint (none) -> Saber_V1:L1305095001400001
- D65: renamed from D71; footprint (none) -> Saber_V1:L1305095001400001
- D66: renamed from D78; footprint (none) -> Saber_V1:L1305095001400001
- D67: renamed from D65; footprint (none) -> Saber_V1:L1305095001400001
- D68: renamed from D72; footprint (none) -> Saber_V1:L1305095001400001
- D69: renamed from D79; footprint (none) -> Saber_V1:L1305095001400001
- D70: renamed from D66; footprint (none) -> Saber_V1:L1305095001400001
- D71: renamed from D73; footprint (none) -> Saber_V1:L1305095001400001
- D72: renamed from D80; footprint (none) -> Saber_V1:L1305095001400001
- D73: renamed from D67; footprint (none) -> Saber_V1:L1305095001400001
- D75: renamed from D81; footprint (none) -> Saber_V1:L1305095001400001
- D76: renamed from D68; footprint (none) -> Saber_V1:L1305095001400001
- D77: renamed from D75; footprint (none) -> Saber_V1:L1305095001400001
- D78: renamed from D82; footprint (none) -> Saber_V1:L1305095001400001
- D79: renamed from D69; footprint (none) -> Saber_V1:L1305095001400001
- D80: renamed from D76; footprint (none) -> Saber_V1:L1305095001400001
- D81: renamed from D83; footprint (none) -> Saber_V1:L1305095001400001
- D82: renamed from D70; footprint (none) -> Saber_V1:L1305095001400001
- D83: renamed from D77; footprint (none) -> Saber_V1:L1305095001400001
- D85: value L130-5095001400001 -> COB Filament LED; footprint (none) -> Connector_PinHeader_2.54mm:PinHeader_1x02_P2.54mm_Vertical
Connections:
- net GND: now also R11.2, R12.2, R15.2, R16.2, R19.2, R20.2, R23.2, R24.2, R27.2, R28.2, R3.2, R4.2, R7.2, R8.2; no longer D12.1 (K), D21.1 (K), D24.1 (K), D33.1 (K), D36.1 (K), D45.1 (K), D48.1 (K), D57.1 (K), D60.1 (K), D69.1 (K), D72.1 (K), D81.1 (K), D84.1 (K), D9.1 (K)
- net at D60.2 (A): now also D59.1 (K); no longer R20.2
- net at R20.1: now also D60.1 (K); no longer D59.1 (K)
- net at D8.1 (K): now also D9.2 (A); no longer R3.1
- net at R4.1: now also D12.1 (K); no longer D11.1 (K)
- net at D12.2 (A): now also D11.1 (K); no longer R4.2
- net at D21.2 (A): now also D20.1 (K); no longer R7.2
- net at D69.2 (A): now also D68.1 (K); no longer R23.2
- net at R11.1: now also D33.1 (K); no longer D32.1 (K)
- net at D33.2 (A): now also D32.1 (K); no longer R11.2
- net at R12.1: now also D36.1 (K); no longer D35.1 (K)
- net at D36.2 (A): now also D35.1 (K); no longer R12.2
- net at R16.1: now also D48.1 (K); no longer D47.1 (K)
- net at D48.2 (A): now also D47.1 (K); no longer R16.2
- net at D80.1 (K): now also D81.2 (A); no longer R27.1
- net at R7.1: now also D21.1 (K); no longer D20.1 (K)
- net at R15.1: now also D45.1 (K); no longer D44.1 (K)
- net at D45.2 (A): now also D44.1 (K); no longer R15.2
- net at D57.2 (A): now also D56.1 (K); no longer R19.2
- net at D24.2 (A): now also D23.1 (K); no longer R8.2
- net at D84.2 (A): now also D83.1 (K); no longer R28.2
- net at R19.1: now also D57.1 (K); no longer D56.1 (K)
- net at R8.1: now also D24.1 (K); no longer D23.1 (K)
- net at D72.2 (A): now also D71.1 (K); no longer R24.2
- net at R23.1: now also D69.1 (K); no longer D68.1 (K)
- net at R24.1: now also D72.1 (K); no longer D71.1 (K)
- net at R28.1: now also D84.1 (K); no longer D83.1 (K)
- new net: D9.1 (K), R3.1
- new net: D81.1 (K), R27.1
Other:
- moved on the sheet: D12, D21, D24, D33, D36, D45, D48, D57, D60, D69, D72, D81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
