File: Electrical/01c_V4 - Powered Platters/02_Basic 2D Platter_V2/00_PCB Designs/PoweredPlatter2_LED Blade_V1/PoweredPlatter2_LED Blade_V1.kicad_sch (KiCad schematic)
At the start: 0 parts

Commit message: adding LED Blade for Powered Platter 2. PCBs are being milled, 3D print needs to still be designed
Parts:
- added D1, D2, D3, D4, D5, D6, D7: LED_3mm, LED_THT:LED_D3.0mm, symbol Device:LED
- added J1: Conn_01x08, Connector_PinHeader_2.54mm:PinHeader_1x08_P2.54mm_Vertical, symbol Connector_Generic:Conn_01x08
- added R1, R2, R3, R4, R5, R6, R7: 300ohm_0603, Resistor_SMD:R_0603_1608Metric_Pad0.98x0.95mm_HandSolder, symbol Device:R_US
Connections:
- new net: D2.2 (A), R2.2
- new net: D7.2 (A), R7.2
- new net: D4.2 (A), R4.2
- new net: D1.2 (A), R1.2
- new net: D3.2 (A), R3.2
- new net: D6.2 (A), R6.2
- new net: D5.2 (A), R5.2
- new net GND: D1.1 (K), D2.1 (K), D3.1 (K), D4.1 (K), D5.1 (K), D6.1 (K), D7.1 (K), J1.8 (Pin_8)
- new net pixel1: J1.1 (Pin_1), R1.1
- new net pixel2: J1.2 (Pin_2), R2.1
- new net pixel3: J1.3 (Pin_3), R3.1
- new net pixel4: J1.4 (Pin_4), R4.1
- new net pixel5: J1.5 (Pin_5), R5.1
- new net pixel6: J1.6 (Pin_6), R6.1
- new net pixel7: J1.7 (Pin_7), R7.1
Other:
- note added: "LEDs and their resistors connected to the Powered Zoetrope platter Designed to interface with Pixel Platter V2 3mm through hole LEDs arranged in a row close to eachother"
